File: C64.sch (KiCad schematic (older format))
At the start: 238 parts, among them CN1 Keyboard, CN10 JP2E, CN2 USERPORT-C64-EDGE, CN3 CASSETTEPORT, CN4 DIN6, CN5 DIN5, CN6 EXPANSIONPORT, CN7 MAB7SH, CN8 CONTROL_PORT, CN9 CONTROL_PORT, J1 Conn_01x01, J2 Conn_01x01, J3 Conn_01x01, Q1 TIP29B, Q2 2N4401, Q3 2N3904, Q4 PN2222, Q5 PN2222, Q6 PN2222, Q7 PN2222, Q8 PN2222, SW1 DPDT_SWITCH, U1 6526, U10 4164, U11 4164, U12 4164, U13 SN74257N, U14 SN74258N, U15 SN74139N, U16 4066, U17 C64PLA, U18 6581, U19 6569, U2 6526, U20 556DIGITAL, U21 4164, U22 4164, U23 4164, U24 4164, U25 SN74257N, U26 74373N, U27 SN7408N, U28 4066, U29 SN7474N, U3 2364, U30 SN74193N, U31 SN74629, U32 MC4044, U4 2364, U5 2332, U6 2114, U7 6510, U8 SN7406NN, U9 4164, Y1 17.73 MHz

Commit message: added ground and vcc fill area's
also adjusted a bit on schematic to make it match board
Parts:
- removed CN7: MAB7SH, cn7:MAB7SH, symbol C64-eagle-import:MAB7SH
- added CN7: DIN7, DIN7:DIN7, symbol DIN7
Connections:
- wire segments 1602 -> 1617
Other:
- moved on the sheet: CR6

Commit message: cleaned up the outer edge
Parts:
- CN2: footprint userport:UPS24EDGE -> USERPORT:USERPORT
Changed lines of the file:
@@
 	11900 20100 11800 20100
 Wire Wire Line
-	11800 20400 11800 20100
+	11800 20100 11800 20400
 Wire Wire Line
 	11900 20300 11800 20300
 Wire Wire Line
-	10400 20400 11800 20400
+	11800 20400 10400 20400
 Wire Wire Line
 	10800 20400 10800 20300
@@
 	5600 6400 4900 6400
 Wire Wire Line
-	4600 7100 4900 6400
+	4900 6400 4600 7100
 Wire Wire Line
-	3300 7100 4600 7100
+	4600 7100 3300 7100
 Wire Wire Line
 	3500 4500 4000 4500
@@
 	5600 12700 4400 12700
 Wire Wire Line
-	4400 13500 4400 12700
+	4400 12700 4400 13500
 Wire Wire Line
-	2400 13500 4400 13500
+	4400 13500 2400 13500
 Wire Wire Line
 	3700 12600 3700 13500
@@
 	5600 12600 4300 12600
 Wire Wire Line
-	4300 13400 4300 12600
+	4300 12600 4300 13400
 Wire Wire Line
-	2400 13400 4300 13400
+	4300 13400 2400 13400
 Wire Wire Line
 	3400 12600 3400 13400
@@
 	5100 11800 4000 11800
 Wire Wire Line
-	4000 13000 4000 11800
+	4000 11800 4000 13000
 Wire Wire Line
-	2400 13000 4000 13000
+	4000 13000 2400 13000
 Wire Wire Line
 	2800 12600 2800 13100
@@
 	5200 11900 4100 11900
 Wire Wire Line
-	4100 13100 4100 11900
+	4100 11900 4100 13100
 Wire Wire Line
-	2400 13100 4100 13100
+	4100 13100 2400 13100
 Connection ~ 7900 17300
 Connection ~ 5300 15000
@@
 	14000 14800 14000 14100
 Wire Wire Line
-	16500 14100 14000 14100
+	14000 14100 16500 14100
 Wire Wire Line
-	16500 10600 16500 14100
+	16500 14100 16500 10600
 Wire Wire Line
 	16500 10700 15400 10700
@@
 	13900 14000 16400 14000
 Wire Wire Line
-	16400 10800 16400 14000
+	16400 14000 16400 10800
 Wire Wire Line
-	15400 10800 16400 10800
+	16400 10800 15400 10800
 Wire Wire Line
 	16300 10600 16300 10800
@@
 	21200 6900 21300 6900
 Wire Wire Line
-	21300 6500 21300 6900
+	21300 6900 21300 6500
 Wire Wire Line
 	8200 6500 24700 6500
@@
 	15400 11300 15800 11300
 Wire Wire Line
-	15800 13100 15800 11300
+	15800 11300 15800 13100
 Wire Wire Line
-	12700 13100 15800 13100
+	15800 13100 12700 13100
 Wire Wire Line
 	12700 13100 12700 13000
@@
 	8400 12100 8000 12100
 Wire Wire Line
-	8000 9700 8000 12100
+	8000 12100 8000 9700
 Wire Wire Line
 	1800 9900 2300 9900
@@
 	24400 8900 24900 8900
 Wire Wire Line
-	24900 7600 24900 8900
+	24900 8900 24900 7600
 Wire Wire Line
-	22100 7600 24900 7600
+	24900 7600 22100 7600
 Wire Wire Line
 	22100 7600 22100 12300
@@
 F 0 "CN2" H 1500 15020 59  0000 L BNN
 F 1 "USERPORT-C64-EDGE" H 1500 12700 59  0000 L BNN
-F 2 "userport:UPS24EDGE" H 1900 13900 50  0001 C CNN
+F 2 "USERPORT:USERPORT" H 1900 13900 50  0001 C CNN
 F 3 "" H 1900 13900 50  0001 C CNN
 	1    1900 13900
@@
 	19100 8900 19100 15200
 Wire Bus Line
-	11200 3700 11200 6100
+	11200 6100 11200 3700
 Wire Bus Line
 	22600 6300 22600 10400

Commit message: more adjustment to schematic
~56 unconnected left. most inside the vic area
Connections:
- net labels removed: N$150, N$166
- wire segments 1617 -> 1620
Changed lines of the file:
@@
 Wire Wire Line
 	7100 6200 6800 6200
-Text Label 19500 9200 0    70   ~ 0
+Text Label 19500 9000 0    70   ~ 0
 D1
 Wire Wire Line
@@
 Wire Wire Line
 	7100 6300 6800 6300
-Text Label 19500 9000 0    70   ~ 0
+Text Label 19500 9100 0    70   ~ 0
 D2
 Wire Wire Line
@@
 Wire Wire Line
 	7100 6400 6800 6400
-Text Label 19500 9100 0    70   ~ 0
+Text Label 19500 9200 0    70   ~ 0
 D3
 Wire Wire Line
@@
 	7600 13500 6800 13500
 Wire Wire Line
-	10600 9700 11300 9700
+	10600 9700 11500 9700
 Wire Wire Line
 	11300 9700 11300 12900
@@
 Connection ~ 11100 13500
 Connection ~ 15900 13500
-Connection ~ 13700 13500
 Wire Wire Line
 	11050 11000 11100 11000
@@
 	14300 15100 13700 15100
 Wire Wire Line
-	13700 15100 13700 13500
+	13700 15100 13700 13600
 Connection ~ 7900 13600
 Connection ~ 25000 5500
@@
 Text Label 13600 13500 0    10   ~ 0
 PHI2
-Text Label 14250 15100 0    10   ~ 0
-PHI2
 Text Label 6900 13900 0    10   ~ 0
 NMI
@@
 Text Label 14150 15300 0    10   ~ 0
 N$165
-Text Label 14200 15400 0    10   ~ 0
-N$166
 Text Label 14150 15500 0    10   ~ 0
 N$135
@@
 Text Label 16800 14250 0    10   ~ 0
 N$54
-Text Label 16450 10000 0    10   ~ 0
-N$150
 Text Label 23100 12900 0    10   ~ 0
 PHI2
-Text Label 23100 13100 0    10   ~ 0
-N$150
 Text Label 23100 13500 0    10   ~ 0
 RW
@@
 Wire Wire Line
 	5050 19850 5050 19300
+Connection ~ 13700 13600
+Text Label 13650 13600 0    10   ~ 0
+RW
+Connection ~ 13700 13500
+Text Label 14200 15100 0    10   ~ 0
+RW
+Text Label 14150 15400 0    10   ~ 0
+RES
+Wire Wire Line
+	16500 10000 16500 9400
+Wire Wire Line
+	16500 9400 11500 9400
+Wire Wire Line
+	11500 9400 11500 9700
+Connection ~ 11300 9700
+Connection ~ 16500 10000
+Text Label 23100 13100 0    10   ~ 0
+RES
+Text Label 16450 10000 0    10   ~ 0
+RES
 $EndSCHEMATC

Commit message: a few more adjustmenst
~55 unconnected left
Connections:
- wire segments 1620 -> 1622
Changed lines of the file:
@@
 	5300 19000 5300 19060
 Wire Wire Line
-	4400 19000 4400 18700
-Wire Wire Line
-	4400 18700 900  18700
+	900  18700 4700 18700
 Wire Wire Line
 	900  18700 900  14100
@@
 	1000 18600 6100 18600
 Wire Wire Line
-	4800 18600 4800 19700
-Wire Wire Line
 	6900 17900 6100 17900
 Wire Wire Line
@@
 	18100 10000 18100 13100
 Wire Wire Line
-	18100 10000 16400 10000
+	16400 10000 18100 10000
 Wire Wire Line
 	15400 11100 16200 11100
@@
 Text Label 4600 17400 0    10   ~ 0
 N$58
-Text Label 6800 17900 0    10   ~ 0
-N$24
-Text Label 4900 18600 0    10   ~ 0
-N$24
-Text Label 1050 14200 0    10   ~ 0
+Text Label 1100 14100 0    10   ~ 0
 N$24
-Text Label 4500 19000 0    10   ~ 0
-N$23
-Text Label 1000 14100 0    10   ~ 0
+Text Label 4850 19000 0    10   ~ 0
 N$23
 Text Label 5300 19050 0    10   ~ 0
@@
 Text Label 16450 10000 0    10   ~ 0
 RES
+Wire Wire Line
+	4800 18600 4800 19000
+Connection ~ 4800 19000
+Wire Wire Line
+	4700 18700 4700 19450
+Wire Wire Line
+	4700 19450 4800 19450
+Wire Wire Line
+	4800 19450 4800 19700
+Text Label 4900 18600 0    10   ~ 0
+N$23
+Text Label 6800 17900 0    10   ~ 0
+N$23
+Text Label 1100 14200 0    10   ~ 0
+N$23
 $EndSCHEMATC

Commit message: last updates etc
Time to take a break :-D
Connections:
- net labels added: +5vc
- wire segments 1622 -> 1621
- no-connect marks 0 -> 22
