File: C64.sch (KiCad schematic (older format))
At the start: 238 parts, among them CN1 Keyboard, CN10 JP2E, CN2 USERPORT-C64-EDGE, CN3 CASSETTEPORT, CN4 DIN6, CN5 DIN5, CN6 EXPANSIONPORT, CN7 DIN7, CN8 CONTROL_PORT, CN9 CONTROL_PORT, J1 Conn_01x01, J2 Conn_01x01, J3 Conn_01x01, Q1 TIP29B, Q2 2N4401, Q3 2N3904, Q4 PN2222, Q5 PN2222, Q6 PN2222, Q7 PN2222, Q8 PN2222, SW1 DPDT_SWITCH, U1 6526, U10 4164, U11 4164, U12 4164, U13 SN74257N, U14 SN74258N, U15 SN74139N, U16 4066, U17 C64PLA, U18 6581, U19 6569, U2 6526, U20 556DIGITAL, U21 4164, U22 4164, U23 4164, U24 4164, U25 SN74257N, U26 74373N, U27 SN7408N, U28 4066, U29 SN7474N, U3 2364, U30 SN74193N, U31 SN74629, U32 MC4044, U4 2364, U5 2332, U6 2114, U7 6510, U8 SN7406NN, U9 4164, Y1 17.73 MHz

Commit message: 4 connections left
There should be a via under R46 but the 2 traks that cross each other does not have the same name

Have checked the RES line and it all seems to connect, there must be a microscopic disconnect somewhere on the RES line

Next step is to import all holes on one of the user layers and check that all via's are there
Parts:
- removed R48: 300, Resistor:12_03_07, symbol C64-eagle-import:R-EU_0204_2V
- removed R50: 1 M, Resistor:12_03_07, symbol C64-eagle-import:R-EU_0204_2V
Connections:
- net labels removed: N$43
- wire segments 1621 -> 1614
- no-connect marks 22 -> 23

Commit message: 2 connections left
C34 and Via under R46 is the mystery

will need to check that all via's are in place, one missing and it can fail
Connections:
- net labels added: N$166

Commit message: corrected a few more things
Thanks to Fredric QJ Blåholtz for the help so far
Parts:
- C93: value 1000 F -> 1000 pF
Connections:
- net labels removed: N$25
Other:
- moved on the sheet: C34, C49, R46

Commit message: added u33 and u34 on schematic
these needs to be wired by the tracks on the board. no schematic found with them wired in
Parts:
- added U33: 7402, symbol 7402
- added U34: 74LS175, symbol 74LS175
Changed lines of the file:
@@
 LIBS:DIN7
 LIBS:BRIDGE_RECTIFIER
+LIBS:74xx
 LIBS:C64-cache
 EELAYER 25 0
@@
 	11900 20100 11800 20100
 Wire Wire Line
-	11800 20400 11800 20100
+	11800 20100 11800 20400
 Wire Wire Line
-	10400 20400 11800 20400
+	11800 20400 10400 20400
 Wire Wire Line
 	10800 20400 10800 20300
@@
 	5600 6400 4900 6400
 Wire Wire Line
-	4600 7100 4900 6400
+	4900 6400 4600 7100
 Wire Wire Line
-	3300 7100 4600 7100
+	4600 7100 3300 7100
 Wire Wire Line
 	3500 4500 4000 4500
@@
 	5600 12700 4400 12700
 Wire Wire Line
-	4400 13500 4400 12700
+	4400 12700 4400 13500
 Wire Wire Line
-	2400 13500 4400 13500
+	4400 13500 2400 13500
 Wire Wire Line
 	3700 12600 3700 13500
@@
 	5600 12600 4300 12600
 Wire Wire Line
-	4300 13400 4300 12600
+	4300 12600 4300 13400
 Wire Wire Line
-	2400 13400 4300 13400
+	4300 13400 2400 13400
 Wire Wire Line
 	3400 12600 3400 13400
@@
 	5100 11800 4000 11800
 Wire Wire Line
-	4000 13000 4000 11800
+	4000 11800 4000 13000
 Wire Wire Line
-	2400 13000 4000 13000
+	4000 13000 2400 13000
 Wire Wire Line
 	2800 12600 2800 13100
@@
 	5200 11900 4100 11900
 Wire Wire Line
-	4100 13100 4100 11900
+	4100 11900 4100 13100
 Wire Wire Line
-	2400 13100 4100 13100
+	4100 13100 2400 13100
 Connection ~ 7900 17300
 Connection ~ 5300 15000
@@
 	14000 14800 14000 14100
 Wire Wire Line
-	16500 14100 14000 14100
+	14000 14100 16500 14100
 Wire Wire Line
-	16500 10600 16500 14100
+	16500 14100 16500 10600
 Wire Wire Line
 	16500 10700 15400 10700
@@
 	13900 14000 16400 14000
 Wire Wire Line
-	16400 10800 16400 14000
+	16400 14000 16400 10800
 Wire Wire Line
-	15400 10800 16400 10800
+	16400 10800 15400 10800
 Wire Wire Line
 	16300 10600 16300 10800
@@
 	21200 6900 21300 6900
 Wire Wire Line
-	21300 6500 21300 6900
+	21300 6900 21300 6500
 Wire Wire Line
 	8200 6500 24700 6500
@@
 	15400 11300 15800 11300
 Wire Wire Line
-	15800 13100 15800 11300
+	15800 11300 15800 13100
 Wire Wire Line
-	12700 13100 15800 13100
+	15800 13100 12700 13100
 Wire Wire Line
 	12700 13100 12700 13000
@@
 	8400 12100 8000 12100
 Wire Wire Line
-	8000 9700 8000 12100
+	8000 12100 8000 9700
 Wire Wire Line
 	1800 9900 2300 9900
@@
 	24400 8900 24900 8900
 Wire Wire Line
-	24900 7600 24900 8900
+	24900 8900 24900 7600
 Wire Wire Line
-	22100 7600 24900 7600
+	24900 7600 22100 7600
 Wire Wire Line
 	22100 7600 22100 12300
@@
 	19100 8900 19100 15200
 Wire Bus Line
-	11200 3700 11200 6100
+	11200 6100 11200 3700
 Wire Bus Line
 	22600 6300 22600 10400
@@
 	28600 16300 28600 16200
 $Comp
-L C64-eagle-import:+9V #V?
+L C64-eagle-import:+9V #V0176
 U 1 0 5A9B4796
 P 5900 20000
-F 0 "#V?" H 5900 20000 50  0001 C CNN
+F 0 "#V0176" H 5900 20000 50  0001 C CNN
 F 1 "+9V" H 5825 20125 59  0000 L BNN
 F 2 "" H 5900 20000 50  0001 C CNN
@@
 Text Label 5050 19400 0    10   ~ 0
 +9V
+$Comp
+L 7402 U33
+U 1 1 5A9BA328
+P 22150 18200
+F 0 "U33" H 22150 18250 50  0000 C CNN
+F 1 "7402" H 22200 18150 50  0000 C CNN
+F 2 "" H 22150 18200 50  0001 C CNN
+F 3 "" H 22150 18200 50  0001 C CNN
+	1    22150 18200
+	1    0    0    -1
+$EndComp
+$Comp
+L 7402 U33
+U 2 1 5A9BA5FD
+P 22150 18900
+F 0 "U33" H 22150 18950 50  0000 C CNN
+F 1 "7402" H 22200 18850 50  0000 C CNN
+F 2 "" H 22150 18900 50  0001 C CNN
+F 3 "" H 22150 18900 50  0001 C CNN
+	2    22150 18900
+	1    0    0    -1
+$EndComp
+$Comp
+L 7402 U33
+U 3 1 5A9BA886
+P 22150 19650
+F 0 "U33" H 22150 19700 50  0000 C CNN
+F 1 "7402" H 22200 19600 50  0000 C CNN
+F 2 "" H 22150 19650 50  0001 C CNN
+F 3 "" H 22150 19650 50  0001 C CNN
+	3    22150 19650
+	1    0    0    -1
+$EndComp
+$Comp
+L 7402 U33
+U 4 1 5A9BAB81
+P 22200 20350
+F 0 "U33" H 22200 20400 50  0000 C CNN
+F 1 "7402" H 22250 20300 50  0000 C CNN
+F 2 "" H 22200 20350 50  0001 C CNN
+F 3 "" H 22200 20350 50  0001 C CNN
+	4    22200 20350
+	1    0    0    -1
+$EndComp
+$Comp
+L 74LS175 U34
+U 1 1 5A9BAE24
+P 23800 19250
+F 0 "U34" H 23800 19250 50  0000 C CNN
+F 1 "74LS175" H 23900 18850 50  0000 C CNN
+F 2 "" H 23800 19250 50  0001 C CNN
+F 3 "" H 23800 19250 50  0001 C CNN
+	1    23800 19250
+	1    0    0    -1
+$EndComp
 $EndSCHEMATC
