File: C64.sch (KiCad schematic (older format))
At the start: 239 parts, among them CN1 Keyboard, CN10 JP2E, CN2 USERPORT-C64-EDGE, CN3 CASSETTEPORT, CN4 DIN6, CN5 DIN5, CN6 EXPANSIONPORT, CN7 DIN7, CN8 CONTROL_PORT, CN9 CONTROL_PORT, J1 Conn_01x01, J2 Conn_01x01, J3 Conn_01x01, Q1 TIP29B, Q2 2N4401, Q3 2N3904, Q4 PN2222, Q5 PN2222, Q6 PN2222, Q7 PN2222, Q8 PN2222, SW1 DPDT_SWITCH, U1 6526, U10 4164, U11 4164, U12 4164, U13 SN74257N, U14 SN74258N, U15 SN74139N, U16 4066, U17 C64PLA, U18 6581, U19 6569, U2 6526, U20 556DIGITAL, U21 4164, U22 4164, U23 4164, U24 4164, U25 SN74257N, U26 74373N, U27 SN7408N, U28 4066, U29 SN7474N, U3 2364, U30 SN74193N, U31 SN74629, U32 MC4044, U33 7402, U34 74LS175, U4 2364, U5 2332, U6 2114, U7 6510, U8 SN7406NN, U9 4164, Y1 17.73 MHz

Commit message: added 2 missing ic's
these are for NTSC versions
Parts:
- removed U33: 7402, symbol 7402
- added U33: 74LS02, Housings_DIP:DIP-14_W7.62mm, symbol 74LS02
- U34: footprint (none) -> SN74629:SN74629
- U34: renamed from U?; footprint (none) -> SN74629:SN74629
Connections:
- wire segments 1616 -> 1651
Other:
- note added: "? Ends blind\non board"
- note added: "Based on schematic done by Ruud Baltissen.\nValues and footprints corrected by Bo Herrmannsen\nHelp with correcting schematic to match board by Fredric QJ Blåholtz"
- note removed: "Based on schematic done by Ruud Baltissen.\nValues and footprints corrected by Bo Herrmannsen"
- moved on the sheet: U34B
Changed lines of the file:
@@
 LIBS:BRIDGE_RECTIFIER
 LIBS:74ls175
+LIBS:74ls02
 LIBS:C64-cache
 EELAYER 25 0
@@
 	1    0    0    -1
 $EndComp
-Text Notes 26650 21850 0    59   ~ 0
-Based on schematic done by Ruud Baltissen.\nValues and footprints corrected by Bo Herrmannsen
+Text Notes 26650 21750 0    59   ~ 0
+Based on schematic done by Ruud Baltissen.\nValues and footprints corrected by Bo Herrmannsen\nHelp with correcting schematic to match board by Fredric QJ Blåholtz
 $Comp
 L c64_lib:Keyboard CN1
@@
 +9V
 $Comp
-L 7402 U33
-U 1 1 5A9BA328
-P 22150 18200
-F 0 "U33" H 22150 18250 50  0000 C CNN
-F 1 "7402" H 22200 18150 50  0000 C CNN
-F 2 "" H 22150 18200 50  0001 C CNN
-F 3 "" H 22150 18200 50  0001 C CNN
-	1    22150 18200
-	1    0    0    -1
-$EndComp
-$Comp
-L 7402 U33
-U 2 1 5A9BA5FD
-P 22150 18900
-F 0 "U33" H 22150 18950 50  0000 C CNN
-F 1 "7402" H 22200 18850 50  0000 C CNN
-F 2 "" H 22150 18900 50  0001 C CNN
-F 3 "" H 22150 18900 50  0001 C CNN
-	2    22150 18900
-	1    0    0    -1
-$EndComp
-$Comp
-L 7402 U33
-U 3 1 5A9BA886
-P 22150 19650
-F 0 "U33" H 22150 19700 50  0000 C CNN
-F 1 "7402" H 22200 19600 50  0000 C CNN
-F 2 "" H 22150 19650 50  0001 C CNN
-F 3 "" H 22150 19650 50  0001 C CNN
-	3    22150 19650
-	1    0    0    -1
-$EndComp
-$Comp
-L 7402 U33
-U 4 1 5A9BAB81
-P 22200 20350
-F 0 "U33" H 22200 20400 50  0000 C CNN
-F 1 "7402" H 22250 20300 50  0000 C CNN
-F 2 "" H 22200 20350 50  0001 C CNN
-F 3 "" H 22200 20350 50  0001 C CNN
-	4    22200 20350
-	1    0    0    -1
-$EndComp
-$Comp
 L 74LS175 U34
 U 1 1 5A9C0D5D
@@
 F 0 "U34" H 23800 20600 50  0000 C CNN
 F 1 "74LS175" H 23900 20200 50  0000 C CNN
-F 2 "" H 23800 20600 50  0001 C CNN
+F 2 "SN74629:SN74629" H 23800 20600 50  0001 C CNN
 F 3 "" H 23800 20600 50  0001 C CNN
 	1    23800 20600
@@
 $EndComp
 $Comp
-L 74LS175 U?
+L 74LS175 U34
 U 2 1 5A9CD34F
 P 28950 2000
-F 0 "U?" H 28950 2000 50  0000 C CNN
+F 0 "U34" H 28950 2000 50  0000 C CNN
 F 1 "74LS175" H 29050 1600 50  0001 C CNN
-F 2 "" H 28950 2000 50  0001 C CNN
+F 2 "SN74629:SN74629" H 28950 2000 50  0001 C CNN
 F 3 "" H 28950 2000 50  0001 C CNN
 	2    28950 2000
-	-1   0    0    1
+	1    0    0    -1
 $EndComp
 Wire Bus Line
@@
 	28600 16300 28600 16200
 $Comp
-L C64-eagle-import:GND #GND?
+L C64-eagle-import:GND #GND0177
 U 1 0 5A9CFF2D
 P 28950 2700
-F 0 "#GND?" H 28950 2700 50  0001 C CNN
+F 0 "#GND0177" H 28950 2700 50  0001 C CNN
 F 1 "GND" H 28850 2600 59  0000 L BNN
 F 2 "" H 28950 2700 50  0001 C CNN
@@
 	1    0    0    -1
 $EndComp
+Wire Wire Line
+	28950 1400 28950 1600
+Wire Wire Line
+	28950 2400 28950 2600
+Text Label 28950 2550 0    10   ~ 0
+GND
+$Comp
+L 74LS02 U33
+U 1 1 5AA1406D
+P 21450 18750
+F 0 "U33" H 21425 18725 59  0000 L BNN
+F 1 "74LS02" H 21150 18450 59  0001 L BNN
+F 2 "Housings_DIP:DIP-14_W7.62mm" H 21450 18750 50  0001 C CNN
+F 3 "" H 21450 18750 50  0001 C CNN
+	1    21450 18750
+	1    0    0    -1
+$EndComp
+$Comp
+L 74LS02 U33
+U 2 1 5AA1432C
+P 21450 19350
+F 0 "U33" H 21425 19325 59  0000 L BNN
+F 1 "74LS02" H 21150 19050 59  0001 L BNN
+F 2 "Housings_DIP:DIP-14_W7.62mm" H 21450 19350 50  0001 C CNN
+F 3 "" H 21450 19350 50  0001 C CNN
+	2    21450 19350
+	1    0    0    -1
+$EndComp
+$Comp
+L 74LS02 U33
+U 3 1 5AA145C7
+P 21450 19950
+F 0 "U33" H 21425 19925 59  0000 L BNN
+F 1 "74LS02" H 21150 19650 59  0001 L BNN
+F 2 "Housings_DIP:DIP-14_W7.62mm" H 21450 19950 50  0001 C CNN
+F 3 "" H 21450 19950 50  0001 C CNN
+	3    21450 19950
+	1    0    0    -1
+$EndComp
+$Comp
+L 74LS02 U33
+U 4 1 5AA14872
+P 21450 20550
+F 0 "U33" H 21425 20525 59  0000 L BNN
+F 1 "74LS02" H 21150 20250 59  0001 L BNN
+F 2 "Housings_DIP:DIP-14_W7.62mm" H 21450 20550 50  0001 C CNN
+F 3 "" H 21450 20550 50  0001 C CNN
+	4    21450 20550
+	1    0    0    -1
+$EndComp
+$Comp
+L 74LS02 U33
+U 5 1 5AA15CD2
+P 28600 2000
+F 0 "U33" H 28575 1975 59  0000 L BNN
+F 1 "74LS02" H 28300 1700 59  0001 L BNN
+F 2 "Housings_DIP:DIP-14_W7.62mm" H 28600 2000 50  0001 C CNN
+F 3 "" H 28600 2000 50  0001 C CNN
+	5    28600 2000
+	1    0    0    -1
+$EndComp
+$Comp
+L C64-eagle-import:VCC #V0178
+U 1 0 5AA2231A
+P 28600 1300
+F 0 "#V0178" H 28600 1300 50  0001 C CNN
+F 1 "VCC" H 28525 1425 59  0000 L BNN
+F 2 "" H 28600 1300 50  0001 C CNN
+F 3 "" H 28600 1300 50  0001 C CNN
+	1    28600 1300
+	-1   0    0    -1
+$EndComp
+Text Label 28600 1500 0    10   ~ 0
+VCC
+Wire Wire Line
+	28600 1400 28600 1600
+$Comp
+L C64-eagle-import:GND #GND0179
+U 1 0 5AA236E0
+P 28600 2700
+F 0 "#GND0179" H 28600 2700 50  0001 C CNN
+F 1 "GND" H 28500 2600 59  0000 L BNN
+F 2 "" H 28600 2700 50  0001 C CNN
+F 3 "" H 28600 2700 50  0001 C CNN
+	1    28600 2700
+	1    0    0    -1
+$EndComp
+Text Label 28600 2500 0    10   ~ 0
+GND
+Wire Wire Line
+	28600 2400 28600 2600
 $Comp
-L C64-eagle-import:+5V_2 #V?
-U 1 0 5A9D02C5
+L C64-eagle-import:VCC #V0180
+U 1 0 5AA2859A
 P 28950 1300
-F 0 "#V?" H 28950 1300 50  0001 C CNN
-F 1 "+5Vc" H 28800 1425 59  0000 L BNN
+F 0 "#V0180" H 28950 1300 50  0001 C CNN
+F 1 "VCC" H 28875 1425 59  0000 L BNN
 F 2 "" H 28950 1300 50  0001 C CNN
 F 3 "" H 28950 1300 50  0001 C CNN
 	1    28950 1300
-	1    0    0    -1
+	-1   0    0    -1
 $EndComp
+Text Label 28950 1500 0    10   ~ 0
+VCC
 Wire Wire Line
-	28950 1400 28950 1550
+	20950 18850 20450 18850
 Wire Wire Line
-	28950 2500 28950 2600
-Text Label 28950 1450 0    10   ~ 0
-+5vc
-Text Label 28950 2550 0    10   ~ 0
+	20950 20450 20450 20450
+Text Label 20750 18850 0    10   ~ 0
+N$155
+Text Label 20700 20450 0    10   ~ 0
+N$155
+$Comp
+L C64-eagle-import:GND #GND0181
+U 1 0 5AA35D7B
+P 22350 19450
+F 0 "#GND0181" H 22350 19450 50  0001 C CNN
+F 1 "GND" H 22250 19350 59  0000 L BNN
+F 2 "" H 22350 19450 50  0001 C CNN
+F 3 "" H 22350 19450 50  0001 C CNN
+	1    22350 19450
+	1    0    0    -1
+$EndComp
+Wire Wire Line
+	21950 19350 22350 19350
+Text Label 22100 19350 0    10   ~ 0
 GND
+Wire Wire Line
+	20950 18650 20950 18400
+Wire Wire Line
+	20950 18400 22700 18400
+Wire Wire Line
+	22700 18400 22700 21050
+Wire Wire Line
+	22700 21050 23100 21050
+Wire Wire Line
+	23100 20200 22700 20200
+Connection ~ 22700 20200
+Wire Wire Line
+	20950 19250 20650 19250
+Wire Wire Line
+	20650 19250 20650 19850
+Wire Wire Line
+	20650 19850 20950 19850
+Wire Wire Line
+	20650 19650 22400 19650
+Wire Wire Line
+	22400 19650 22400 20950
+Wire Wire Line
+	22400 20950 23100 20950
+Connection ~ 20650 19650
+Text Label 20850 19450 0    10   ~ 0
+PHI0
+Wire Wire Line
+	20950 19450 20750 19450
+Wire Wire Line
+	20950 20650 20950 21000
+Wire Wire Line
+	20950 21000 22250 21000
+Wire Wire Line
+	22250 21000 22250 19950
+Wire Wire Line
+	22250 19950 21950 19950
+Wire Wire Line
+	20450 20450 20450 18850
+Text Notes 20500 20100 0    60   ~ 0
+? Ends blind\non board
+Wire Wire Line
+	21950 20550 21950 21800
+Wire Wire Line
+	21950 21800 25100 21800
+Wire Wire Line
+	25100 21800 25100 20650
+Wire Wire Line
+	25100 20650 24500 20650
+Wire Wire Line
+	24500 20150 24500 19850
+Wire Wire Line
+	24500 19850 22900 19850
+Wire Wire Line
+	22900 19850 22900 20350
+Wire Wire Line
+	22900 20350 23100 20350
+Wire Wire Line
+	24500 20350 24900 20350
+Wire Wire Line
+	24900 20350 24900 21700
+Wire Wire Line
+	24900 21700 22800 21700
+Wire Wire Line
+	22800 21700 22800 20550
+Wire Wire Line
+	22800 20550 23100 20550
 $EndSCHEMATC

Commit message: added 3d shapes to ntsc chips
Parts:
- U33: footprint Housings_DIP:DIP-14_W7.62mm -> 7402:7402
Changed lines of the file:
@@
 F 0 "U33" H 21425 18725 59  0000 L BNN
 F 1 "74LS02" H 21150 18450 59  0001 L BNN
-F 2 "Housings_DIP:DIP-14_W7.62mm" H 21450 18750 50  0001 C CNN
+F 2 "7402:7402" H 21450 18750 50  0001 C CNN
 F 3 "" H 21450 18750 50  0001 C CNN
 	1    21450 18750
@@
 F 0 "U33" H 21425 19325 59  0000 L BNN
 F 1 "74LS02" H 21150 19050 59  0001 L BNN
-F 2 "Housings_DIP:DIP-14_W7.62mm" H 21450 19350 50  0001 C CNN
+F 2 "7402:7402" H 21450 19350 50  0001 C CNN
 F 3 "" H 21450 19350 50  0001 C CNN
 	2    21450 19350
@@
 F 0 "U33" H 21425 19925 59  0000 L BNN
 F 1 "74LS02" H 21150 19650 59  0001 L BNN
-F 2 "Housings_DIP:DIP-14_W7.62mm" H 21450 19950 50  0001 C CNN
+F 2 "7402:7402" H 21450 19950 50  0001 C CNN
 F 3 "" H 21450 19950 50  0001 C CNN
 	3    21450 19950
@@
 F 0 "U33" H 21425 20525 59  0000 L BNN
 F 1 "74LS02" H 21150 20250 59  0001 L BNN
-F 2 "Housings_DIP:DIP-14_W7.62mm" H 21450 20550 50  0001 C CNN
+F 2 "7402:7402" H 21450 20550 50  0001 C CNN
 F 3 "" H 21450 20550 50  0001 C CNN
 	4    21450 20550
@@
 F 0 "U33" H 28575 1975 59  0000 L BNN
 F 1 "74LS02" H 28300 1700 59  0001 L BNN
-F 2 "Housings_DIP:DIP-14_W7.62mm" H 28600 2000 50  0001 C CNN
+F 2 "7402:7402" H 28600 2000 50  0001 C CNN
 F 3 "" H 28600 2000 50  0001 C CNN
 	5    28600 2000

Commit message: all tracks connected. Hurra :-D
Connections:
- wire segments 1651 -> 1658
Changed lines of the file:
@@
 Text Label 10700 10100 0    10   ~ 0
 IRQ
-Text Label 10750 10300 0    10   ~ 0
-N$168
 Text Label 10750 10500 0    10   ~ 0
 N$168
@@
 	1    0    0    -1
 $EndComp
+$Comp
+L C64-eagle-import:GND #GND0177
+U 1 0 5A9CFF2D
+P 28950 2700
+F 0 "#GND0177" H 28950 2700 50  0001 C CNN
+F 1 "GND" H 28850 2600 59  0000 L BNN
+F 2 "" H 28950 2700 50  0001 C CNN
+F 3 "" H 28950 2700 50  0001 C CNN
+	1    28950 2700
+	1    0    0    -1
+$EndComp
+Text Label 28950 2550 0    10   ~ 0
+GND
+$Comp
+L C64-eagle-import:VCC #V0178
+U 1 0 5AA2231A
+P 28600 1300
+F 0 "#V0178" H 28600 1300 50  0001 C CNN
+F 1 "VCC" H 28525 1425 59  0000 L BNN
+F 2 "" H 28600 1300 50  0001 C CNN
+F 3 "" H 28600 1300 50  0001 C CNN
+	1    28600 1300
+	-1   0    0    -1
+$EndComp
+Text Label 28600 1500 0    10   ~ 0
+VCC
+$Comp
+L C64-eagle-import:GND #GND0179
+U 1 0 5AA236E0
+P 28600 2700
+F 0 "#GND0179" H 28600 2700 50  0001 C CNN
+F 1 "GND" H 28500 2600 59  0000 L BNN
+F 2 "" H 28600 2700 50  0001 C CNN
+F 3 "" H 28600 2700 50  0001 C CNN
+	1    28600 2700
+	1    0    0    -1
+$EndComp
+Text Label 28600 2500 0    10   ~ 0
+GND
+$Comp
+L C64-eagle-import:VCC #V0180
+U 1 0 5AA2859A
+P 28950 1300
+F 0 "#V0180" H 28950 1300 50  0001 C CNN
+F 1 "VCC" H 28875 1425 59  0000 L BNN
+F 2 "" H 28950 1300 50  0001 C CNN
+F 3 "" H 28950 1300 50  0001 C CNN
+	1    28950 1300
+	-1   0    0    -1
+$EndComp
+Text Label 28950 1500 0    10   ~ 0
+VCC
+Text Label 20750 18850 0    10   ~ 0
+N$155
+Text Label 21850 20550 0    10   ~ 0
+N$155
+$Comp
+L C64-eagle-import:GND #GND0181
+U 1 0 5AA35D7B
+P 20600 19350
+F 0 "#GND0181" H 20600 19350 50  0001 C CNN
+F 1 "GND" H 20500 19250 59  0000 L BNN
+F 2 "" H 20600 19350 50  0001 C CNN
+F 3 "" H 20600 19350 50  0001 C CNN
+	1    20600 19350
+	1    0    0    -1
+$EndComp
+Text Label 20750 19250 0    10   ~ 0
+GND
+Text Label 20850 19450 0    10   ~ 0
+PHI0
+Text Notes 20500 20100 0    60   ~ 0
+? Ends blind\non board
+$Comp
+L 74LS02 U33
+U 1 1 5AA46F15
+P 21350 18750
+F 0 "U33" H 21325 18725 59  0000 L BNN
+F 1 "74LS02" H 21050 18450 59  0001 L BNN
+F 2 "7402:7402" H 21350 18750 50  0001 C CNN
+F 3 "" H 21350 18750 50  0001 C CNN
+	1    21350 18750
+	1    0    0    -1
+$EndComp
+$Comp
+L 74LS02 U33
+U 5 1 5AA4E7C5
+P 28600 2000
+F 0 "U33" H 28575 1975 59  0000 L BNN
+F 1 "74LS02" H 28300 1700 59  0001 L BNN
+F 2 "7402:7402" H 28600 2000 50  0001 C CNN
+F 3 "" H 28600 2000 50  0001 C CNN
+	5    28600 2000
+	1    0    0    -1
+$EndComp
+$Comp
+L 74LS02 U33
+U 4 1 5AA476CC
+P 21350 20550
+F 0 "U33" H 21325 20525 59  0000 L BNN
+F 1 "74LS02" H 21050 20250 59  0001 L BNN
+F 2 "7402:7402" H 21350 20550 50  0001 C CNN
+F 3 "" H 21350 20550 50  0001 C CNN
+	4    21350 20550
+	1    0    0    -1
+$EndComp
+$Comp
+L 74LS02 U33
+U 3 1 5AA47437
+P 21350 19950
+F 0 "U33" H 21325 19925 59  0000 L BNN
+F 1 "74LS02" H 21050 19650 59  0001 L BNN
+F 2 "7402:7402" H 21350 19950 50  0001 C CNN
+F 3 "" H 21350 19950 50  0001 C CNN
+	3    21350 19950
+	1    0    0    -1
+$EndComp
+$Comp
+L 74LS02 U33
+U 2 1 5AA471AE
+P 21350 19350
+F 0 "U33" H 21325 19325 59  0000 L BNN
+F 1 "74LS02" H 21050 19050 59  0001 L BNN
+F 2 "7402:7402" H 21350 19350 50  0001 C CNN
+F 3 "" H 21350 19350 50  0001 C CNN
+	2    21350 19350
+	1    0    0    -1
+$EndComp
 Wire Bus Line
 	24400 3300 24400 3900
@@
 Wire Wire Line
 	28600 16300 28600 16200
-$Comp
-L C64-eagle-import:GND #GND0177
-U 1 0 5A9CFF2D
-P 28950 2700
-F 0 "#GND0177" H 28950 2700 50  0001 C CNN
-F 1 "GND" H 28850 2600 59  0000 L BNN
-F 2 "" H 28950 2700 50  0001 C CNN
-F 3 "" H 28950 2700 50  0001 C CNN
-	1    28950 2700
-	1    0    0    -1
-$EndComp
 Wire Wire Line
 	28950 1400 28950 1600
 Wire Wire Line
 	28950 2400 28950 2600
-Text Label 28950 2550 0    10   ~ 0
-GND
-$Comp
-L 74LS02 U33
-U 1 1 5AA1406D
-P 21450 18750
-F 0 "U33" H 21425 18725 59  0000 L BNN
-F 1 "74LS02" H 21150 18450 59  0001 L BNN
-F 2 "7402:7402" H 21450 18750 50  0001 C CNN
-F 3 "" H 21450 18750 50  0001 C CNN
-	1    21450 18750
-	1    0    0    -1
-$EndComp
-$Comp
-L 74LS02 U33
-U 2 1 5AA1432C
-P 21450 19350
-F 0 "U33" H 21425 19325 59  0000 L BNN
-F 1 "74LS02" H 21150 19050 59  0001 L BNN
-F 2 "7402:7402" H 21450 19350 50  0001 C CNN
-F 3 "" H 21450 19350 50  0001 C CNN
-	2    21450 19350
-	1    0    0    -1
-$EndComp
-$Comp
-L 74LS02 U33
-U 3 1 5AA145C7
-P 21450 19950
-F 0 "U33" H 21425 19925 59  0000 L BNN
-F 1 "74LS02" H 21150 19650 59  0001 L BNN
-F 2 "7402:7402" H 21450 19950 50  0001 C CNN
-F 3 "" H 21450 19950 50  0001 C CNN
-	3    21450 19950
-	1    0    0    -1
-$EndComp
-$Comp
-L 74LS02 U33
-U 4 1 5AA14872
-P 21450 20550
-F 0 "U33" H 21425 20525 59  0000 L BNN
-F 1 "74LS02" H 21150 20250 59  0001 L BNN
-F 2 "7402:7402" H 21450 20550 50  0001 C CNN
-F 3 "" H 21450 20550 50  0001 C CNN
-	4    21450 20550
-	1    0    0    -1
-$EndComp
-$Comp
-L 74LS02 U33
-U 5 1 5AA15CD2
-P 28600 2000
-F 0 "U33" H 28575 1975 59  0000 L BNN
-F 1 "74LS02" H 28300 1700 59  0001 L BNN
-F 2 "7402:7402" H 28600 2000 50  0001 C CNN
-F 3 "" H 28600 2000 50  0001 C CNN
-	5    28600 2000
-	1    0    0    -1
-$EndComp
-$Comp
-L C64-eagle-import:VCC #V0178
-U 1 0 5AA2231A
-P 28600 1300
-F 0 "#V0178" H 28600 1300 50  0001 C CNN
-F 1 "VCC" H 28525 1425 59  0000 L BNN
-F 2 "" H 28600 1300 50  0001 C CNN
-F 3 "" H 28600 1300 50  0001 C CNN
-	1    28600 1300
-	-1   0    0    -1
-$EndComp
-Text Label 28600 1500 0    10   ~ 0
-VCC
 Wire Wire Line
 	28600 1400 28600 1600
-$Comp
-L C64-eagle-import:GND #GND0179
-U 1 0 5AA236E0
-P 28600 2700
-F 0 "#GND0179" H 28600 2700 50  0001 C CNN
-F 1 "GND" H 28500 2600 59  0000 L BNN
-F 2 "" H 28600 2700 50  0001 C CNN
-F 3 "" H 28600 2700 50  0001 C CNN
-	1    28600 2700
-	1    0    0    -1
-$EndComp
-Text Label 28600 2500 0    10   ~ 0
-GND
 Wire Wire Line
 	28600 2400 28600 2600
-$Comp
-L C64-eagle-import:VCC #V0180
-U 1 0 5AA2859A
-P 28950 1300
-F 0 "#V0180" H 28950 1300 50  0001 C CNN
-F 1 "VCC" H 28875 1425 59  0000 L BNN
-F 2 "" H 28950 1300 50  0001 C CNN
-F 3 "" H 28950 1300 50  0001 C CNN
-	1    28950 1300
-	-1   0    0    -1
-$EndComp
-Text Label 28950 1500 0    10   ~ 0
-VCC
 Wire Wire Line
 	20950 18850 20450 18850
 Wire Wire Line
 	20950 20450 20450 20450
-Text Label 20750 18850 0    10   ~ 0
-N$155
-Text Label 20700 20450 0    10   ~ 0
-N$155
-$Comp
-L C64-eagle-import:GND #GND0181
-U 1 0 5AA35D7B
-P 22350 19450
-F 0 "#GND0181" H 22350 19450 50  0001 C CNN
-F 1 "GND" H 22250 19350 59  0000 L BNN
-F 2 "" H 22350 19450 50  0001 C CNN
-F 3 "" H 22350 19450 50  0001 C CNN
-	1    22350 19450
-	1    0    0    -1
-$EndComp
-Wire Wire Line
-	21950 19350 22350 19350
-Text Label 22100 19350 0    10   ~ 0
-GND
-Wire Wire Line
-	20950 18650 20950 18400
 Wire Wire Line
-	20950 18400 22700 18400
+	21850 18400 22700 18400
 Wire Wire Line
 	22700 18400 22700 21050
@@
 Connection ~ 22700 20200
 Wire Wire Line
-	20950 19250 20650 19250
-Wire Wire Line
-	20650 19250 20650 19850
+	20650 19850 20650 20200
 Wire Wire Line
 	20650 19850 20950 19850
 Wire Wire Line
-	20650 19650 22400 19650
+	22000 19650 22400 19650
 Wire Wire Line
 	22400 19650 22400 20950
 Wire Wire Line
 	22400 20950 23100 20950
-Connection ~ 20650 19650
-Text Label 20850 19450 0    10   ~ 0
-PHI0
 Wire Wire Line
 	20950 19450 20750 19450
@@
 	20950 21000 22250 21000
 Wire Wire Line
-	22250 21000 22250 19950
+	22250 21000 22250 20200
 Wire Wire Line
-	22250 19950 21950 19950
-Wire Wire Line
-	20450 20450 20450 18850
-Text Notes 20500 20100 0    60   ~ 0
-? Ends blind\non board
+	20450 20450 20450 21150
 Wire Wire Line
-	21950 20550 21950 21800
+	21950 21150 21950 21800
 Wire Wire Line
 	21950 21800 25100 21800
@@
 Wire Wire Line
 	22800 20550 23100 20550
+Wire Wire Line
+	21850 20550 21950 20550
+Wire Wire Line
+	21850 18750 21850 18400
+Connection ~ 21850 18400
+Wire Wire Line
+	20950 19250 20600 19250
+Wire Wire Line
+	21850 19350 22000 19350
+Wire Wire Line
+	22000 19350 22000 19950
+Connection ~ 22000 19650
+Wire Wire Line
+	22250 20200 20650 20200
+Connection ~ 20650 19850
+Connection ~ 22250 20200
+Wire Wire Line
+	22000 19950 21850 19950
+Wire Wire Line
+	20450 21150 21950 21150
+Connection ~ 20450 20450
+Connection ~ 21950 21150
+Wire Wire Line
+	20450 18850 20450 20300
+Wire Wire Line
+	20450 20300 21950 20300
+Wire Wire Line
+	21950 20300 21950 20550
+Text Label 10700 10300 0    10   ~ 0
+NMI
 $EndSCHEMATC

Commit message: minor corrections
Connections:
- net labels removed: N$58
- wire segments 1658 -> 1659
Other:
- moved on the sheet: U33C
Changed lines of the file:
@@
 	-1   0    0    1
 $EndComp
-Text Label 5800 17450 0    10   ~ 0
-N$58
 Text Label 12900 10000 0    10   ~ 0
 N$169
@@
 Text Label 20750 18850 0    10   ~ 0
 N$155
-Text Label 21850 20550 0    10   ~ 0
-N$155
 $Comp
 L C64-eagle-import:GND #GND0181
@@
 Text Label 20850 19450 0    10   ~ 0
 PHI0
-Text Notes 20500 20100 0    60   ~ 0
+Text Notes 21850 19900 0    60   ~ 0
 ? Ends blind\non board
 $Comp
@@
 L 74LS02 U33
 U 3 1 5AA47437
-P 21350 19950
-F 0 "U33" H 21325 19925 59  0000 L BNN
-F 1 "74LS02" H 21050 19650 59  0001 L BNN
-F 2 "7402:7402" H 21350 19950 50  0001 C CNN
-F 3 "" H 21350 19950 50  0001 C CNN
-	3    21350 19950
+P 21350 19850
+F 0 "U33" H 21325 19825 59  0000 L BNN
+F 1 "74LS02" H 21050 19550 59  0001 L BNN
+F 2 "7402:7402" H 21350 19850 50  0001 C CNN
+F 3 "" H 21350 19850 50  0001 C CNN
+	3    21350 19850
 	1    0    0    -1
 $EndComp
@@
 Connection ~ 22700 20200
 Wire Wire Line
-	20650 19850 20650 20200
-Wire Wire Line
-	20650 19850 20950 19850
+	20650 19750 20950 19750
 Wire Wire Line
 	22000 19650 22400 19650
@@
 	20950 19450 20750 19450
 Wire Wire Line
-	20950 20650 20950 21000
-Wire Wire Line
-	20950 21000 22250 21000
-Wire Wire Line
-	22250 21000 22250 20200
+	22250 20550 22250 20200
 Wire Wire Line
 	20450 20450 20450 21150
@@
 	22800 20550 23100 20550
 Wire Wire Line
-	21850 20550 21950 20550
-Wire Wire Line
 	21850 18750 21850 18400
 Connection ~ 21850 18400
@@
 	21850 19350 22000 19350
 Wire Wire Line
-	22000 19350 22000 19950
+	22000 19350 22000 20150
 Connection ~ 22000 19650
 Wire Wire Line
 	22250 20200 20650 20200
-Connection ~ 20650 19850
 Connection ~ 22250 20200
 Wire Wire Line
-	22000 19950 21850 19950
+	22000 20150 20950 20150
 Wire Wire Line
 	20450 21150 21950 21150
@@
 	20450 18850 20450 20300
 Wire Wire Line
-	20450 20300 21950 20300
-Wire Wire Line
-	21950 20300 21950 20550
+	20450 20300 20700 20300
 Text Label 10700 10300 0    10   ~ 0
 NMI
+$Comp
+L C64-eagle-import:GND #GND0182
+U 1 0 5A9B8D13
+P 20300 18750
+F 0 "#GND0182" H 20300 18750 50  0001 C CNN
+F 1 "GND" H 20200 18650 59  0000 L BNN
+F 2 "" H 20300 18750 50  0001 C CNN
+F 3 "" H 20300 18750 50  0001 C CNN
+	1    20300 18750
+	1    0    0    -1
+$EndComp
+Wire Wire Line
+	20950 18650 20300 18650
+Text Label 20700 18650 0    10   ~ 0
+GND
+Wire Wire Line
+	20650 20200 20650 19750
+Wire Wire Line
+	20950 20150 20950 19950
+Text Label 20750 20650 0    10   ~ 0
+N$155
+Wire Wire Line
+	20700 20300 20700 20650
+Wire Wire Line
+	20700 20650 20950 20650
+Wire Wire Line
+	22250 20550 21850 20550
+Text Label 5900 17450 0    10   ~ 0
+RES
 $EndSCHEMATC

Commit message: more adjustments
Parts:
- renumbered Q3 to Q1, Q1 to Q3
Changed lines of the file:
@@
 $EndComp
 $Comp
-L TIP29B Q1
+L TIP29B Q3
 U 1 1 5AC0169F
 P 10200 17200
-F 0 "Q1" H 10150 17000 59  0000 L BNN
-F 1 "TIP29B" V 10200 17450 59  0000 L BNN
+F 0 "Q3" H 10150 17000 59  0000 L BNN
+F 1 "TIP29B" V 10400 17100 59  0000 L BNN
 F 2 "TIP29B:TIP29B" H 10200 17200 50  0001 C CNN
 F 3 "" H 10200 17200 50  0001 C CNN
@@
 $EndComp
 $Comp
-L 2N3904 Q3
+L 2N3904 Q1
 U 1 1 5AC02BDC
 P 10500 16800
-F 0 "Q3" H 10600 16800 59  0000 L BNN
+F 0 "Q1" H 10600 16800 59  0000 L BNN
 F 1 "2N3904" V 10050 16350 59  0000 L BNN
 F 2 "TO92:TO92" H 10500 16800 50  0001 C CNN
@@
 P 11200 17100
 F 0 "Q2" H 11250 17100 59  0000 L BNN
-F 1 "2N4401" V 12400 16850 59  0000 L BNN
+F 1 "2N4401" V 12150 17250 59  0000 L BNN
 F 2 "TO92:TO92" H 11200 17100 50  0001 C CNN
 F 3 "" H 11200 17100 50  0001 C CNN

Commit message: first adjustments on silk screen
Parts:
- Q1: value 2N3904 -> 2N4401; symbol 2N3904 -> 2N4401
- Q2: value 2N4401 -> 2N3904; symbol 2N4401 -> 2N3904
Changed lines of the file:
@@
 $EndComp
 $Comp
-L 2N3904 Q1
+L 2N4401 Q1
 U 1 1 5AC02BDC
 P 10500 16800
 F 0 "Q1" H 10600 16800 59  0000 L BNN
-F 1 "2N3904" V 10050 16350 59  0000 L BNN
+F 1 "2N4401" V 10800 16650 59  0000 L BNN
 F 2 "TO92:TO92" H 10500 16800 50  0001 C CNN
 F 3 "" H 10500 16800 50  0001 C CNN
@@
 $EndComp
 $Comp
-L 2N4401 Q2
+L 2N3904 Q2
 U 1 1 5AC04462
 P 11200 17100
 F 0 "Q2" H 11250 17100 59  0000 L BNN
-F 1 "2N4401" V 12150 17250 59  0000 L BNN
+F 1 "2N3904" V 11450 16950 59  0000 L BNN
 F 2 "TO92:TO92" H 11200 17100 50  0001 C CNN
 F 3 "" H 11200 17100 50  0001 C CNN
