File: C64.sch (KiCad schematic (older format))
At the start: 238 parts, among them CN1 Keyboard, CN10 JP2E, CN2 USERPORT-C64-EDGE, CN3 CASSETTEPORT, CN4 DIN6, CN5 DIN5, CN6 EXPANSIONPORT, CN7 DIN7, CN8 CONTROL_PORT, CN9 CONTROL_PORT, J1 Conn_01x01, J2 Conn_01x01, J3 Conn_01x01, Q1 2N4401, Q2 2N3904, Q3 TIP29B, Q4 PN2222, Q5 PN2222, Q6 PN2222, Q7 PN2222, Q8 PN2222, SW1 DPDT_SWITCH, U1 6526, U10 4164, U11 4164, U12 4164, U13 SN74257N, U14 SN74258N, U15 SN74139N, U16 4066, U17 C64PLA, U18 6581, U19 6569, U2 6526, U20 556DIGITAL, U21 4164, U22 4164, U23 4164, U24 4164, U25 SN74257N, U26 74373N, U27 SN7408N, U28 4066, U29 SN7474N, U3 2364, U30 SN74193N, U31 SN74629, U32 MC4044, U33 74LS02, U34 74LS175, U4 2364, U5 2332, U6 2114, U7 6510, U8 SN7406NN, U9 4164, Y1 17.73 MHz

Commit message: more footprints and schematic corrections
a lot of the schematic symbols was still from the eagle import and pcb footprints had not been saved as individual footprints
Parts:
- removed CN1: Keyboard, 20way:20way, symbol c64_lib:Keyboard
- removed CN2: USERPORT-C64-EDGE, USERPORT:USERPORT, symbol C64-eagle-import:USERPORT-C64-EDGE
- removed CN3: CASSETTEPORT, CASSETTEPORT:CASSETTEPORT, symbol C64-eagle-import:CASSETTEPORT
- removed CN4: DIN6, cn4:DIN6, symbol C64-eagle-import:DIN6
- removed CN5: DIN5, cn5:DIN5, symbol C64-eagle-import:DIN5
- removed CN6: EXPANSIONPORT, EXPANSIONPORT:EXPANSIONPORT, symbol C64-eagle-import:EXPANSIONPORT-C64
- removed CN8, CN9: CONTROL_PORT, Controlport:CONTROL_PORT, symbol C64-eagle-import:CONTROL_PORT
- removed FB1, FB10, FB11, FB12, FB18, FB2, FB3, FB4, FB5, FB6: FB_0307/12R_0307/12, 12_3_07:12_03_07, symbol c64_lib:FB-12_3_7
- removed FB13: FERRIT, 12_3_07:12_03_07, symbol c64_lib:FB-12_3_7
- removed FB14, FB15, FB16, FB17: FB_0307/12R_0307/12, 12_3_07:12_03_07, symbol C64-eagle-import:FB_0307_12R_0307_12
- removed FB7, FB8, FB9: FB_12_3_7, 12_3_07:12_03_07, symbol c64_lib:FB-12_3_7
- removed L1, L2: 2.2 uH, INDUCTOR_P12:12_03_07, symbol C64-eagle-import:INDUCTOR_12_3_7
- removed L3: 3 uH, INDUCTOR_P12:12_03_07, symbol C64-eagle-import:INDUCTOR_12_3_7
- removed L4: LINEFILTER, linefilter:LINEFILTER, symbol C64-eagle-import:LINEFILTER
- removed L5: 1.2 uH, INDUCTOR_P15:P15, symbol C64-eagle-import:COIL
- removed R25: 1 K Trim Pot, symbol C64-eagle-import:POT_METER
- removed R27: 2 K Trim Pot, symbol C64-eagle-import:POT_METER
- removed RF1: RF-MODULATOR, rfmodulator:RF-MODULATOR, symbol C64-eagle-import:RF-MODULATOR
- removed RP1, RP2: 33, RESISTOR_PACK_4:RESISTOR_PACK_4, symbol c64_lib:RP4
- removed RP3: RP8, RESISTOR_PACK_4:RESISTOR_PACK_4, symbol c64_lib:RP8
- removed RP4: 3.3 K, RESISTOR_PACK_9:RESISTOR_PACK_9, symbol c64_lib:RP9
- removed SW1: DPDT_SWITCH, switch:DPDT_SWITCH, symbol C64-eagle-import:DPDT_SWITCH
- removed U26: 74373N, 74373N:74373N, symbol c64_lib:74373N
- removed VR1: VR, 7812:7812, symbol c64_lib:VR
- removed VR2: VR, 7805:7805, symbol c64_lib:VR
- removed Y1: 17.73 MHz, Crystal:HC49TL-H, symbol C64-eagle-import:HC49TL-H
- added CN1: KEYBOARD, 20way:20way, symbol KEYBOARD
- added CN2: USERPORT, USERPORT:USERPORT, symbol USERPORT
- added CN3: CASSETTEPORT, CASSETTEPORT:CASSETTEPORT, symbol CASSETTEPORT
- added CN4: DIN6, DIN6:DIN6, symbol DIN6
- added CN5: DIN5, DIN5:DIN5, symbol DIN5
- added CN6: EXPANSIONPORT, EXPANSIONPORT:EXPANSIONPORT, symbol EXPANSIONPORT
- added CN8, CN9: CONTROL_PORT, CONTROL_PORT:CONTROL_PORT, symbol CONTROL_PORT
- added FB1, FB10, FB11, FB12, FB13, FB14, FB15, FB16, FB17, FB18, FB2, FB3, FB4, FB5, FB6, FB7, FB8, FB9: FERRITE_BEAD, FERRITE_BEAD:FERRITE_BEAD, symbol FERRITE_BEAD
- added L1, L2: 2.2 uH, INDUCTOR_P12:12_03_07, symbol INDUCTOR
- added L3: 3 uH, INDUCTOR_P12:12_03_07, symbol INDUCTOR
- added L4: LINEFILTER, symbol LINEFILTER
- added L5: 1.2 uH, INDUCTOR_P15:P15, symbol INDUCTOR
- added R25: 1 K Trim Pot, POT_METER:POT_METER, symbol POT_METER
- added R27: 2 K Trim Pot, POT_METER:POT_METER, symbol POT_METER
- added RF1: RF-MODULATOR, RF-MODULATOR:RF-MODULATOR, symbol RF-MODULATOR
- added RP1, RP2: 33, RESISTOR_PACK_4:RESISTOR_PACK_4, symbol RP4
- added RP3: 3.3 K, RESISTOR_PACK_4:RESISTOR_PACK_4, symbol RP8
- added RP4: 3.3 K, RESISTOR_PACK_9:RESISTOR_PACK_9, symbol RP9
- added SW1: DPDT_SWITCH, DPDT_SWITCH:DPDT_SWITCH, symbol DPDT_SWITCH
- added U26: SN74373N, 74373N:74373N, symbol SN74373N
- added VR1: 7812, VR:VR, symbol VR
- added VR2: 7805, VR:VR, symbol VR
- added Y1: 17.73 MHz, Crystal:HC49TL-H, symbol CRYSTAL
- CR4: footprint (none) -> BRIDGE_RECTIFIER:BRIDGE_RECTIFIER
Connections:
- wire segments 1659 -> 1665
- no-connect marks 23 -> 22
Other:
- moved on the sheet: C24
