File: C64.kicad_pcb (KiCad board)
At the start: 2 copper layers, 389.2 x 180.3 mm, 258 parts, among them CN1 Keyboard, CN10 JP2E, CN2 USERPORT-C64-EDGE, CN3 CASSETTEPORT, CN4 DIN6, CN5 DIN5, CN6 EXPANSIONPORT, CN7 DIN7, CN8 CONTROL_PORT, CN9 CONTROL_PORT, J1 Conn_01x01, J2 Conn_01x01, J3 Conn_01x01, Q1 2N4401, Q2 2N3904, Q3 TIP29B, Q4 PN2222, Q5 PN2222, Q6 PN2222, Q7 PN2222, Q8 PN2222, SW1 DPDT_SWITCH, U1 6526, U10 4164, U11 4164, U12 4164, U13 SN74257N, U14 SN74258N, U15 SN74139N, U16 4066, U17 C64PLA, U18 6581, U19 6569, U2 6526, U20 556DIGITAL, U21 4164, U22 4164, U23 4164, U24 4164, U25 SN74257N, U26 74373N, U27 SN7408N, U28 4066, U29 SN7474N, U3 2364, U30 SN74193N, U31 SN74629, U32 MC4044, U33 74LS02, U34 74LS175, U4 2364, U5 2332, U6 2114, U7 6510, U8 SN7406NN, U9 4164, Y1 17.73 MHz

Commit message: more footprints and schematic corrections
a lot of the schematic symbols was still from the eagle import and pcb footprints had not been saved as individual footprints
Parts:
- CN1: value Keyboard -> KEYBOARD
- CN2: value USERPORT-C64-EDGE -> USERPORT
- FB1, FB10, FB11, FB12, FB14, FB15, FB16, FB17, FB18, FB2, FB3, FB4, FB5, FB6: value FB_0307/12R_0307/12 -> FERRITE_BEAD
- FB13: value FERRIT -> FERRITE_BEAD
- FB7, FB8, FB9: value FB_12_3_7 -> FERRITE_BEAD
- RP3: value RP8 -> 3.3 K
- U26: value 74373N -> SN74373N
- VR1: value VR -> 7812
- VR2: value VR -> 7805
- moved FB18 12.8 mm to (382.2, 177.7), turned to 0 degrees
- moved FB6 12.8 mm to (282.4, 116.6), turned to 0 degrees
- moved FB17 12.8 mm to (327.0, 171.2), turned to 180 degrees
- moved FB4 12.8 mm to (314.9, 98.3), turned to 180 degrees
- moved FB16 12.7 mm to (334.7, 180.1), turned to 0 degrees
- moved FB3 12.7 mm to (137.5, 67.7), turned to 0 degrees
- moved FB2 12.7 mm to (135.0, 67.7), turned to 180 degrees
- moved FB15 12.7 mm to (275.4, 179.5), turned to 0 degrees
- moved FB1 12.7 mm to (127.4, 63.9), turned to 0 degrees
- moved FB11 12.7 mm to (227.2, 197.3), turned to 90 degrees
- moved FB12 12.7 mm to (248.0, 218.8), turned to 90 degrees
- moved FB5 12.6 mm to (301.5, 102.0), turned to 0 degrees
- moved FB14 12.6 mm to (275.5, 175.6), turned to 0 degrees
Connections:
- CN1 pad 2: Net-(CN1-Pad2) -> (no net)
- FB1 pad 1: /N$176 -> /N$84
- FB1 pad 2: /N$84 -> /N$176
- FB11 pad 1: /N$14 -> /+12V
- FB11 pad 2: /+12V -> /N$14
- FB12 pad 1: /N$35 -> /+12V
- FB12 pad 2: /+12V -> /N$35
- FB14 pad 1: /N$15 -> /N$16
- FB14 pad 2: /N$16 -> /N$15
- FB15 pad 1: /N$37 -> /N$162
- FB15 pad 2: /N$162 -> /N$37
- FB16 pad 1: /N$70 -> /N$66
- FB16 pad 2: /N$66 -> /N$70
- FB17 pad 1: /N$87 -> /N$82
- FB17 pad 2: /N$82 -> /N$87
- FB18 pad 1: /VCC -> /N$109
- FB18 pad 2: /N$109 -> /VCC
- FB2 pad 1: /N$180 -> /N$133
- FB2 pad 2: /N$133 -> /N$180
- FB3 pad 1: /VCC -> /N$173
- FB3 pad 2: /N$173 -> /VCC
- FB4 pad 1: /RES -> /N$153
- FB4 pad 2: /N$153 -> /RES
- FB5 pad 1: /PHI2 -> /N$141
- FB5 pad 2: /N$141 -> /PHI2
- FB6 pad 1: /N$13 -> /VCC
- FB6 pad 2: /VCC -> /N$13
