File: C64.kicad_pcb (KiCad board)
At the start: 2 copper layers, 389.2 x 180.3 mm, 259 parts, among them CN1 KEYBOARD, CN10 JP2E, CN2 USERPORT, CN3 CASSETTEPORT, CN4 DIN6, CN5 DIN5, CN6 EXPANSIONPORT, CN7 DIN7, CN8 CONTROL_PORT, CN9 CONTROL_PORT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

Commit message: added logo to back side
Parts:
- added G***: LOGO, Logo:logo2, F.Cu at (201.0, 215.6)
