File: C64.kicad_pcb (KiCad board)
At the start: 2 copper layers, 389.2 x 180.3 mm, 260 parts, among them CN1 KEYBOARD, CN10 JP2E, CN2 USERPORT, CN3 CASSETTEPORT, CN4 DIN6, CN5 DIN5, CN6 EXPANSIONPORT, CN7 DIN7, CN8 CONTROL_PORT, CN9 CONTROL_PORT, J1 Conn_01x01, J2 Conn_01x01, J3 Conn_01x01, Q1 2N4401, Q2 2N3904, Q3 TIP29B, Q4 PN2222, Q5 PN2222, Q6 PN2222, Q7 PN2222, Q8 PN2222, SW1 DPDT_SWITCH, U1 6526, U10 4164, U11 4164, U12 4164, U13 SN74257N, U14 SN74258N, U15 SN74139N, U16 4066, U17 C64PLA, U18 6581, U19 6569, U2 6526, U20 556DIGITAL, U21 4164, U22 4164, U23 4164, U24 4164, U25 SN74257N, U26 SN74373N, U27 SN7408N, U28 4066, U29 SN7474N, U3 2364, U30 SN74193N, U31 SN74629, U32 MC4044, U33 74LS02, U34 74LS175, U4 2364, U5 2332, U6 2114, U7 6510, U8 SN7406NN, U9 4164, Y1 17.73 MHz

Commit message: bigger holes
Parts:
- moved CN2 1.50 mm to (59.9, 49.8)
- moved CN3 1.50 mm to (133.6, 50.4)
Routing:
- net /N$23: track 549.9 -> 556.9 mm
- net /N$120: track 76.3 -> 83.4 mm
- net /N$119: track 139.0 -> 146.0 mm
- net /VCC: track 3350.7 -> 3357.7 mm, vias 43 -> 42
- net /RES: track 661.9 -> 668.9 mm
- net /N$173: track 45.2 -> 38.4 mm
- net /GND: track 5389.8 -> 5385.7 mm, vias 65 -> 63
- net /N$84: track 27.1 -> 29.2 mm
- net /N$171: track 267.0 -> 268.8 mm
- net /N$27: track 69.1 -> 70.9 mm
- net /N$133: track 30.8 -> 32.5 mm
- net /+9V: track 247.5 -> 245.9 mm
- net /N$172: track 164.7 -> 166.3 mm
Other:
- board size 389.2 x 180.3 mm -> 389.2 x 181.8 mm
