File: _autosave-C64.kicad_pcb (KiCad board)
At the start: 2 copper layers, 389.2 x 180.3 mm, 258 parts, among them CN1 KEYBOARD, CN10 JP2E, CN2 USERPORT, CN3 CASSETTEPORT, CN4 DIN6, CN5 DIN5, CN6 EXPANSIONPORT, CN7 DIN7, CN8 CONTROL_PORT, CN9 CONTROL_PORT, J1 Conn_01x01, J2 Conn_01x01, J3 Conn_01x01, Q1 2N4401, Q2 2N3904, Q3 TIP29B, Q4 PN2222, Q5 PN2222, Q6 PN2222, Q7 PN2222, Q8 PN2222, SW1 DPDT_SWITCH, U1 6526, U10 4164, U11 4164, U12 4164, U13 SN74257N, U14 SN74258N, U15 SN74139N, U16 4066, U17 C64PLA, U18 6581, U19 6569, U2 6526, U20 556DIGITAL, U21 4164, U22 4164, U23 4164, U24 4164, U25 SN74257N, U26 74373N, U27 SN7408N, U28 4066, U29 SN7474N, U3 2364, U30 SN74193N, U31 SN74629, U32 MC4044, U33 74LS02, U34 74LS175, U4 2364, U5 2332, U6 2114, U7 6510, U8 SN7406NN, U9 4164, Y1 17.73 MHz

Commit message: more footprints and schematic corrections
a lot of the schematic symbols was still from the eagle import and pcb footprints had not been saved as individual footprints
Parts:
- RP3: value RP8 -> 3.3 K
- U26: value 74373N -> SN74373N
- VR1: value VR -> 7812
- VR2: value VR -> 7805
Changed lines of the file:
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@@
     (links 1012)
     (no_connects 0)
-    (area 13.328257 44.179474 411.903943 225.668543)
+    (area 14.923819 44.319555 404.290481 224.771201)
     (thickness 1.6)
     (drawings 10681)
@@
       (effects (font (size 1.2065 1.2065) (thickness 0.127)) (justify right top))
     )
-    (fp_text value RP8 (at 0 0 180) (layer F.SilkS) hide
+    (fp_text value "3.3 K" (at 0 0 180) (layer F.SilkS) hide
       (effects (font (size 1.27 1.27) (thickness 0.15)) (justify right top))
     )
@@
       (effects (font (size 1.2065 1.2065) (thickness 0.1016)) (justify right top))
     )
-    (fp_text value 74373N (at 0 0 270) (layer F.SilkS) hide
+    (fp_text value SN74373N (at 0 0 270) (layer F.SilkS) hide
       (effects (font (size 1.27 1.27) (thickness 0.15)))
     )
@@
       (effects (font (size 1.2065 1.2065) (thickness 0.127)) (justify left bottom))
     )
-    (fp_text value VR (at 0 0 180) (layer F.SilkS) hide
+    (fp_text value 7812 (at 0 0 180) (layer F.SilkS) hide
       (effects (font (size 1.27 1.27) (thickness 0.15)))
     )
@@
       (effects (font (size 1.2065 1.2065) (thickness 0.127)) (justify left bottom))
     )
-    (fp_text value VR (at 0 0 90) (layer F.SilkS) hide
+    (fp_text value 7805 (at 0 0 90) (layer F.SilkS) hide
       (effects (font (size 1.27 1.27) (thickness 0.15)))
     )
@@
   (segment (start 307.4416 185.9026) (end 307.4416 195.7832) (width 0.25) (layer F.Cu) (net 60))
   (segment (start 307.4416 195.7832) (end 307.0606 196.088) (width 0.25) (layer F.Cu) (net 60))
-  (segment (start 287.2848 190.8302) (end 287.2848 190.7178) (width 0.25) (layer F.Cu) (net 60))
-  (segment (start 287.2848 190.7178) (end 287.8328 190.1698) (width 0.25) (layer F.Cu) (net 60))
-  (segment (start 287.8328 190.1698) (end 287.8328 186.2836) (width 0.25) (layer F.Cu) (net 60))
-  (segment (start 287.8328 186.2836) (end 287.2486 185.6994) (width 0.25) (layer F.Cu) (net 60))
-  (segment (start 287.2486 185.6994) (end 282.0416 185.6994) (width 0.25) (layer F.Cu) (net 60))
-  (segment (start 282.0416 185.6994) (end 279.5016 183.1594) (width 0.25) (layer F.Cu) (net 60))
   (segment (start 275.1836 183.1594) (end 279.5016 183.1594) (width 0.25) (layer F.Cu) (net 60))
-  (segment (start 279.5016 183.1594) (end 279.8064 183.1594) (width 0.25) (layer F.Cu) (net 60))
-  (segment (start 279.8064 183.1594) (end 281.8638 181.102) (width 0.25) (layer F.Cu) (net 60))
-  (segment (start 281.8638 181.102) (end 281.8638 169.0878) (width 0.25) (layer F.Cu) (net 60))
   (segment (start 291.7698 170.688) (end 291.7698 170.6118) (width 0.25) (layer F.Cu) (net 60))
   (segment (start 291.7698 170.6118) (end 290.2458 169.0878) (width 0.25) (layer F.Cu) (net 60))
-  (segment (start 290.2458 169.0878) (end 281.8638 169.0878) (width 0.25) (layer F.Cu) (net 60))
-  (segment (start 281.8638 169.0878) (end 275.717 169.0878) (width 0.25) (layer F.Cu) (net 60))
   (segment (start 275.5646 171.9326) (end 275.5646 156.845) (width 0.25) (layer F.Cu) (net 60))
   (segment (start 275.5646 156.845) (end 275.844 156.5656) (width 0.25) (layer F.Cu) (net 60))
@@
   (segment (start 143.429 57.5866) (end 142.8242 58.1914) (width 0.25) (layer B.Cu) (net 60) (status 10))
   (segment (start 142.8242 58.1914) (end 142.8242 58.7502) (width 0.25) (layer B.Cu) (net 60))
+  (segment (start 287.2848 190.8302) (end 287.2848 190.7178) (width 0.25) (layer F.Cu) (net 60))
+  (segment (start 287.2848 190.7178) (end 287.8328 190.1698) (width 0.25) (layer F.Cu) (net 60))
+  (segment (start 287.8328 190.1698) (end 287.8328 186.2836) (width 0.25) (layer F.Cu) (net 60))
+  (segment (start 287.8328 186.2836) (end 287.2486 185.6994) (width 0.25) (layer F.Cu) (net 60))
+  (segment (start 287.2486 185.6994) (end 282.0416 185.6994) (width 0.25) (layer F.Cu) (net 60))
+  (segment (start 282.0416 185.6994) (end 279.5016 183.1594) (width 0.25) (layer F.Cu) (net 60))
+  (segment (start 279.5016 183.1594) (end 279.8064 183.1594) (width 0.25) (layer F.Cu) (net 60))
+  (segment (start 279.8064 183.1594) (end 281.8638 181.102) (width 0.25) (layer F.Cu) (net 60))
+  (segment (start 281.8638 181.102) (end 281.8638 169.0878) (width 0.25) (layer F.Cu) (net 60))
+  (segment (start 290.2458 169.0878) (end 281.8638 169.0878) (width 0.25) (layer F.Cu) (net 60))
+  (segment (start 281.8638 169.0878) (end 275.717 169.0878) (width 0.25) (layer F.Cu) (net 60))
   (segment (start 364.998 135.0772) (end 364.998 134.9502) (width 0.25) (layer F.Cu) (net 61))
   (segment (start 367.792 156.972) (end 367.792 136.0424) (width 0.25) (layer B.Cu) (net 61))
@@
   (segment (start 282.5242 182.9308) (end 282.5242 190.5908) (width 0.25) (layer B.Cu) (net 99))
   (segment (start 282.5242 190.5908) (end 282.2848 190.8302) (width 0.25) (layer B.Cu) (net 99))
-  (segment (start 282.7528 183.1594) (end 287.8836 183.1594) (width 0.25) (layer B.Cu) (net 99) (status 20))
   (segment (start 282.4734 182.88) (end 282.5242 182.9308) (width 0.25) (layer B.Cu) (net 99))
   (segment (start 282.5242 182.9308) (end 282.7528 183.1594) (width 0.25) (layer B.Cu) (net 99))
   (segment (start 282.4734 177.6222) (end 282.4734 182.88) (width 0.25) (layer B.Cu) (net 99))
   (segment (start 284.4038 175.6918) (end 282.4734 177.6222) (width 0.25) (layer B.Cu) (net 99))
+  (segment (start 282.7528 183.1594) (end 287.8836 183.1594) (width 0.25) (layer B.Cu) (net 99) (status 20))
   (segment (start 288.1122 175.6918) (end 284.4038 175.6918) (width 0.25) (layer B.Cu) (net 99) (status 10))
   (segment (start 304.1142 190.9826) (end 296.2656 190.9826) (width 0.25) (layer B.Cu) (net 100))
